File: Hardware/Parameter-Board/Parameter-Board-8.brd (EAGLE design)
At the start: 100 x 80 mm, 10 parts

Commit message: move board to the left and make it smaller
Parts:
- moved 1P1 49.5 mm to (11.4, 75.6)
- moved 1P2 49.5 mm to (11.4, 60.3)
- moved 1P3 49.5 mm to (11.4, 45.1)
- moved 1P4 49.5 mm to (11.4, 29.8)
- moved 2P1 49.5 mm to (36.8, 75.6)
- moved 2P2 49.5 mm to (36.8, 60.3)
- moved 2P3 49.5 mm to (36.8, 45.1)
- moved 2P4 49.5 mm to (36.8, 29.8)
- moved MX1 49.5 mm to (36.8, 12.7)
- moved SV1 49.5 mm to (6.35, 10.2)
Other:
- board size 100 x 80 mm -> 50.5 x 80 mm
