File: Hardware/Parameter-Board/Parameter-Board.sch (EAGLE design)
At the start: 22 parts

Commit message: VEE ist die negative Referenzspannung, welche in unserem Fall GND ist. Die Referenz-Voltage des MCU ist hingegen mit AGND verbunden.
Connections:
- net VEE renamed AGND
- net GND: now also MX1P.GND, MX1P.VEE, MX2P.GND, MX2P.VEE
- net VCC: now also MX1P.VCC, MX2P.VCC

Commit message: Das komplette Board wurde neu geroutet, so dass keine Top-Layer-Brücke nötig und die Leiterbahnführung einheitlicher ist
Connections:
- net 1P1: now also MX1A.X5; no longer MX1A.X1
- net 1P2: now also MX1A.X7; no longer MX1A.X6
- net 1P3: now also MX1A.X6; no longer MX1A.X2
- net 2P1: now also MX1A.X2; no longer MX1A.X0
- net 2P2: now also MX1A.X1; no longer MX1A.X7
- net 2P3: now also MX1A.X0; no longer MX1A.X3
- net 2P4: now also MX1A.X3; no longer MX1A.X5
- net 4P3: now also MX2A.X6; no longer MX2A.X4
- net 4P4: now also MX2A.X4; no longer MX2A.X6
- net A: now also SV1.5
Other:
- moved on the sheet: MX1P, MX2P

Commit message: Endgültiges Boardlayout
Parts:
- H1, H2, H3: value MOUNT-PAD-ROUND2.8 -> MOUNT-PAD-ROUND3.2; device holes:MOUNT-PAD-ROUND2.8 -> holes:MOUNT-PAD-ROUND3.2
Connections:
- net 1P2 renamed 7MX1
- removed net 1P1: 1P1.C, MX1A.X5
- removed net 1P3: 1P3.C, MX1A.X6
- removed net 1P4: 1P4.C, MX1A.X4
- removed net 2P1: 2P1.C, MX1A.X2
- removed net 2P2: 2P2.C, MX1A.X1
- removed net 2P3: 2P3.C, MX1A.X0
- removed net 2P4: 2P4.C, MX1A.X3
- removed net 3P1: 3P1.C, MX2A.X2
- removed net 3P2: 3P2.C, MX2A.X1
- removed net 3P3: 3P3.C, MX2A.X0
- removed net 3P4: 3P4.C, MX2A.X3
- removed net 4P1: 4P1.C, MX2A.X5
- removed net 4P2: 4P2.C, MX2A.X7
- removed net 4P3: 4P3.C, MX2A.X6
- removed net 4P4: 4P4.C, MX2A.X4
- new net 0MX1: 2P4.C, MX1A.X0
- new net 0MX2: 4P3.C, MX2A.X0
- new net 1MX1: 2P3.C, MX1A.X1
- new net 1MX2: 4P2.C, MX2A.X1
- new net 2MX1: 2P2.C, MX1A.X2
- new net 2MX2: 4P1.C, MX2A.X2
- new net 3MX1: 1P4.C, MX1A.X3
- new net 3MX2: 4P4.C, MX2A.X3
- new net 4MX1: 1P1.C, MX1A.X4
- new net 4MX2: 3P1.C, MX2A.X4
- new net 5MX1: 1P3.C, MX1A.X5
- new net 5MX2: 3P4.C, MX2A.X5
- new net 6MX1: 2P1.C, MX1A.X6
- new net 6MX2: 3P2.C, MX2A.X6
- new net 7MX2: 3P3.C, MX2A.X7
- net A: no longer SV1.5
- net AGND: now also 2P1.B, 2P2.B, 2P3.B, 2P4.B, 4P1.B, 4P2.B, 4P3.B, 4P4.B, SV1.4; no longer 2P1.A, 2P2.A, 2P3.A, 2P4.A, 4P1.A, 4P2.A, 4P3.A, 4P4.A, SV1.9
- net GND: now also 2P1.A, 2P2.A, 2P3.A, 2P4.A, 4P1.A, 4P2.A, 4P3.A, 4P4.A, SV1.2; no longer 2P1.B, 2P2.B, 2P3.B, 2P4.B, 4P1.B, 4P2.B, 4P3.B, 4P4.B, SV1.4
- net VCC: now also SV1.1; no longer SV1.3
- net X1: now also SV1.3; no longer SV1.2
- net X2: now also SV1.5; no longer SV1.1
Other:
- moved on the sheet: H1, H2, H3, MX1, MX2
