File: Hardware/Parameter-Board/Parameter-Board.brd (EAGLE design)
At the start: 100 x 80 mm, 22 parts

Commit message: Wenn die drei Bahnenden den gleichen Winkel haben, schaut's einfach schöner aus
Routing:
- net C: track 54.6 -> 53.9 mm
Changed lines of the file:
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@@
 <wire x1="27.94" y1="3.81" x2="50.8" y2="3.81" width="0.4064" layer="16"/>
 <wire x1="50.8" y1="5.08" x2="50.8" y2="3.81" width="0.4064" layer="16"/>
-<wire x1="50.8" y1="3.81" x2="78.74" y2="3.81" width="0.4064" layer="16"/>
-<wire x1="78.74" y1="3.81" x2="78.74" y2="5.08" width="0.4064" layer="16"/>
+<wire x1="50.8" y1="3.81" x2="76.2" y2="3.81" width="0.4064" layer="16"/>
+<wire x1="76.2" y1="3.81" x2="77.47" y2="5.08" width="0.4064" layer="16"/>
+<wire x1="77.47" y1="5.08" x2="78.74" y2="5.08" width="0.4064" layer="16"/>
 </signal>
 <signal name="B">
