File: Hardware/Microdrum/Sequenzer/Sequenzer.sch (EAGLE design)
At the start: 20 parts

Commit message: Bohrlöcher
Parts:
- added H1, H2, H3: MOUNT-PAD-ROUND3.2, holes:MOUNT-PAD-ROUND3.2
Changed lines of the file:
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@@
 <layer number="97" name="Info" color="7" fill="1" visible="yes" active="yes"/>
 <layer number="98" name="Guide" color="6" fill="1" visible="yes" active="yes"/>
+<layer number="250" name="Descript" color="7" fill="1" visible="no" active="no"/>
+<layer number="251" name="SMDround" color="7" fill="1" visible="no" active="no"/>
 </layers>
 <schematic xreflabel="%F%N/%S.%C%R" xrefpart="/%S.%C%R">
@@
 <part name="P+1" library="supply1" deviceset="VCC" device=""/>
 <part name="P+18" library="supply1" deviceset="VCC" device=""/>
+<part name="H2" library="holes" deviceset="MOUNT-PAD-ROUND" device="3.2"/>
+<part name="H3" library="holes" deviceset="MOUNT-PAD-ROUND" device="3.2"/>
+<part name="H1" library="holes" deviceset="MOUNT-PAD-ROUND" device="3.2"/>
 </parts>
 <sheets>
@@
 <instance part="P+1" gate="VCC" x="-7.62" y="-25.4" smashed="yes" rot="R270"/>
 <instance part="P+18" gate="VCC" x="73.66" y="-106.68" smashed="yes" rot="R180"/>
+<instance part="H2" gate="G$1" x="-30.48" y="-71.12"/>
+<instance part="H3" gate="G$1" x="-30.48" y="-63.5"/>
+<instance part="H1" gate="G$1" x="-30.48" y="-78.74"/>
 </instances>
 <busses>
