File: Hardware/Microdrum/Sequenzer/Sequenzer.brd (EAGLE design)
At the start: 100 x 59.7 mm, 20 parts

Commit message: Bohrlöcher
Parts:
- added H1, H2, H3: MOUNT-PAD-ROUND3.2, holes:3,2-PAD
Changed lines of the file:
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@@
 <layer number="97" name="Info" color="7" fill="1" visible="no" active="no"/>
 <layer number="98" name="Guide" color="6" fill="1" visible="no" active="no"/>
+<layer number="250" name="Descript" color="7" fill="1" visible="no" active="no"/>
+<layer number="251" name="SMDround" color="7" fill="1" visible="no" active="no"/>
 </layers>
 <board>
@@
 <attribute name="VALUE" x="43.942" y="6.985" size="1.27" layer="27" ratio="10"/>
 </element>
+<element name="H2" library="holes" package="3,2-PAD" value="MOUNT-PAD-ROUND3.2" x="92.71" y="52.07"/>
+<element name="H3" library="holes" package="3,2-PAD" value="MOUNT-PAD-ROUND3.2" x="7.62" y="52.07"/>
+<element name="H1" library="holes" package="3,2-PAD" value="MOUNT-PAD-ROUND3.2" x="66.675" y="7.62"/>
 </elements>
 <signals>
